File: MouseSMDSensorBoard/MouseSMDSensorBoard.kicad_sch (KiCad schematic)
At the start: 14 parts, among them J1 Conn_01x05

Commit message: Updates based on feedback
Parts:
- removed FET1: BSH108,215, Package_TO_SOT_SMD:SOT-23, symbol Transistor_FET:BF545A
- added FET1: PMV45EN2, Package_TO_SOT_SMD:SOT-23_Handsoldering, symbol PB_Library:PMV45EN2
- added TP1, TP2, TP3, TP4: TestPoint, TestPoint:TestPoint_Pad_D1.5mm, symbol Connector:TestPoint
- PD1: renamed from PD2; value VEMD4010X01 -> QSB34; footprint Resistor_SMD:R_0805_2012Metric -> PBFootPrintLibrary:PLCC_2L_Handsoldering
- PD2: renamed from PD3; symbol Device:D_Photo -> Sensor_Optical:BPW40
- TR1: footprint Package_TO_SOT_SMD:SOT-23 -> Package_TO_SOT_SMD:SOT-23_Handsoldering
- renumbered RPullDown1 to R2, RSENSE1 to R4, R2 to R5, R4 to R6
Connections:
- net ADC: now also TP3.1
- net GND: now also TP4.1
- net at R1.2, R2.1, TR1.3 (C): now also FET1.1 (G)
- net at C1.1, LED1.2 (A), R3.2: now also TP1.1
- net at LED1.1 (K): now also FET1.3 (D), TP2.1
- net at R4.1, TR1.1 (B): now also FET1.2 (S)
- net +3.3V renamed Vcc
- net +9V renamed Vbatt
