File: MouseSMDSensorBoard/MouseSMDSensorBoard.kicad_pcb (KiCad board)
At the start: 2 copper layers, 18 x 35 mm, 14 parts, among them J1 Conn_01x05

Commit message: Updates based on feedback
Parts:
- added TP1: TestPoint, TestPoint:TestPoint_Pad_D1.5mm, F.Cu at (134.6, 97.4)
- added TP2: TestPoint, TestPoint:TestPoint_Pad_D1.5mm, F.Cu at (134.6, 93.8)
- added TP3: TestPoint, TestPoint:TestPoint_Pad_D1.5mm, F.Cu at (146.6, 95.8)
- added TP4: TestPoint, TestPoint:TestPoint_Pad_D1.5mm, F.Cu at (147.2, 89.2)
- FET1: value BSH108,215 -> PMV45EN2; footprint Package_TO_SOT_SMD:SOT-23 -> Package_TO_SOT_SMD:SOT-23_Handsoldering
- PD1: renamed from PD2; value VEMD4010X01 -> QSB34; footprint Resistor_SMD:R_0805_2012Metric -> PBFootPrintLibrary:PLCC_2L_Handsoldering
- TR1: footprint Package_TO_SOT_SMD:SOT-23 -> Package_TO_SOT_SMD:SOT-23_Handsoldering
- moved R2 1.75 mm to (138.2, 80.7)
- moved LED1 1.62 mm to (139.9, 91.8)
- moved R1 1.56 mm to (134.8, 80.9)
- moved R3 1.36 mm to (142.4, 81.2)
- moved TR1 1.35 mm to (139.5, 85.5)
- moved R6 1.27 mm to (148.8, 81.2)
- moved C2 1.25 mm to (148.8, 85.2)
- moved R4 1.17 mm to (142.8, 85.8)
- moved FET1 1.05 mm to (135.6, 85.8)
- moved PD2 0.85 mm to (139.8, 103.8)
- moved C1 0.85 mm to (145.9, 81.7)
- moved PD1 0.40 mm to (141.1, 98.4)
- renumbered PD3 to PD2, RPD1 to R2, RSENSE1 to R4, R2 to R5, R4 to R6
Connections:
- net +3.3V renamed Vcc
- net +9V renamed Vbatt
- FET1 pad 1: Net-(FET1-S) -> Net-(FET1-G)
- FET1 pad 2: Net-(FET1-D) -> Net-(FET1-S)
- FET1 pad 3: Net-(FET1-G) -> Net-(FET1-D)
Routing:
- net GND: track 5.93 -> 17.7 mm
- net Net-(LED1-A): track 15.1 -> 26.0 mm
- net Net-(FET1-D): track 6.93 -> 14.5 mm
- net Net-(FET1-G): track 9.03 -> 12.3 mm
- net /ADC: track 40.9 -> 43.6 mm
- net /LED_ON: track 6.44 -> 4.95 mm
- net Vcc: track 6.60 -> 5.44 mm
- net Net-(FET1-S): track 11.9 -> 12.6 mm
Other:
- board text added: "Vb"
- board text added: "Vbatt"
- board text added: "Vcc"
- board text removed: "3v3"
- board text removed: "vBatt"

Commit message: Sort of ready for JLCPCB
Changed lines of the file:
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@@
 	)
 	(gr_text "GND"
-		(at 142 77.05 90)
+		(at 141.87 77.06 90)
 		(layer "B.SilkS")
 		(effects
@@
 	)
 	(gr_text "GND"
-		(at 141 77.05 -90)
+		(at 140.86 77.06 -90)
 		(layer "F.SilkS")
 		(effects
@@
 	)
 	(gr_text "Vb\n"
-		(at 138.4 77.05 270)
+		(at 138.41 77.15 270)
 		(layer "F.SilkS")
 		(effects
