File: MouseLedSensorDaughterBoard/MouseLedSensorDaughterBoard.kicad_pcb (KiCad board)
At the start: 2 copper layers, 13 x 25 mm, 4 parts, among them J2 Conn_01x04

Commit message: Sort of ready for JLCPCB
Parts:
- PD2: value VEMD4010X01 -> QSB34; footprint Diode_SMD:D_0805_2012Metric_Pad1.15x1.40mm_HandSolder -> PBFootPrintLibrary:PLCC_2L_Handsoldering
- PD3: renamed from SEN; footprint LED_THT:LED_D5.0mm -> LED_THT:LED_D5.0mm_Clear
- moved PD3 1.51 mm to (139.7, 104.5)
- renumbered LED to LED1
Routing:
- net /Sen+: track 21.7 -> 25.8 mm
- net /Sen-: track 20.3 -> 21.1 mm
