File: MouseSMDUKMARSAdvancedBoard/MouseSMDUKMARSAdvancedBoard.kicad_pcb (KiCad board)
At the start: 2 copper layers, 80 x 27.3 mm, 33 parts, among them J1 Conn_01x10

Commit message: Updates based on feedback
Parts:
- FET1, FET2: value BSH108,215 -> PMV45EN2; footprint Package_TO_SOT_SMD:SOT-23 -> Package_TO_SOT_SMD:SOT-23_Handsoldering
- J1: moved to B.Cu
- TR1, TR2: footprint Package_TO_SOT_SMD:SOT-23 -> Package_TO_SOT_SMD:SOT-23_Handsoldering
- moved FET2 3.89 mm to (137.4, 133.0), turned to 90 degrees
- moved FET1 3.68 mm to (137.4, 126.8), turned to 90 degrees
- moved R8 3.15 mm to (146.1, 131.8)
- moved R6 3.13 mm to (146.1, 126.9)
- moved TR2 3.03 mm to (142.1, 133.0), turned to 90 degrees
- moved TR1 2.62 mm to (142.0, 126.8), turned to 90 degrees
- moved C1 2.45 mm to (156.1, 138.8)
- moved R3 2.23 mm to (148.4, 127.0)
- moved R5 2.15 mm to (153.8, 138.8)
- moved R4 2.10 mm to (148.3, 131.8)
- moved J1 0.55 mm to (128.6, 147.6), turned to -90 degrees
Connections:
- net +3.3V renamed Vcc
- net +9V renamed Vbatt
- C1 pad 1: Net-(DLED1-A) -> Net-(DLED2-A)
- C2 pad 1: Net-(FLED1-A) -> Net-(FLED2-A)
- DLED2 pad 1: Net-(DLED1-K) -> Net-(DLED1-A)
- DLED2 pad 2: Net-(DLED1-A) -> Net-(DLED2-A)
- FET1 pad 1: Net-(FET1-S) -> Net-(FET1-G)
- FET1 pad 2: Net-(DLED1-K) -> Net-(FET1-S)
- FET1 pad 3: Net-(FET1-G) -> Net-(DLED1-K)
- FET2 pad 1: Net-(FET2-S) -> Net-(FET2-G)
- FET2 pad 2: Net-(FET2-D) -> Net-(FET2-S)
- FET2 pad 3: Net-(FET2-G) -> Net-(FET2-D)
- FLED2 pad 1: Net-(FET2-D) -> Net-(FLED1-A)
- FLED2 pad 2: Net-(FLED1-A) -> Net-(FLED2-A)
- R5 pad 2: Net-(DLED1-A) -> Net-(DLED2-A)
- R7 pad 2: Net-(FLED1-A) -> Net-(FLED2-A)
Routing:
- net Net-(FET2-D): track 112.5 -> 38.6 mm, vias 2 -> 0
- net Net-(DLED1-K): track 39.2 -> 14.3 mm
- net GND: track 22.4 -> 43.1 mm, vias 9 -> 8
- net Net-(FLED2-A): track 0.00 -> 19.2 mm
- net Net-(DLED2-A): track 0.00 -> 11.4 mm
- net Net-(DLED1-A): track 52.5 -> 42.5 mm, vias 3 -> 0
- net Net-(FLED1-A): track 88.6 -> 82.0 mm
- net Net-(LFPD1-C): track 82.5 -> 87.5 mm, vias 3 -> 2
- net Net-(LDPD1-C): track 34.2 -> 37.7 mm, vias 2 -> 1
- net A0_LF: track 44.9 -> 47.7 mm, vias 2 -> 1
- net A2_LD: track 30.9 -> 28.5 mm
- net A3_RF: track 38.0 -> 39.8 mm, vias 2 -> 1
- net Net-(FET2-G): track 19.4 -> 17.7 mm
- net Net-(FET2-S): track 8.27 -> 9.21 mm
- net Vcc: track 9.08 -> 9.63 mm
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Other:
- board text added: "Vbatt"
- board text added: "Vcc"
- board text removed: "+3.3"
- board text removed: "+9v"

Commit message: Sort of ready for JLCPCB
Parts:
- added H1: 3.2mm, MountingHole:MountingHole_3.2mm_M3_Pad, F.Cu at (115.9, 144.9)
- added H2: 3.2mm, MountingHole:MountingHole_3.2mm_M3_Pad, F.Cu at (164.2, 144.8)
- moved J1 0.89 mm to (128.0, 146.9)
- moved R15 0.28 mm to (125.0, 144.9)
- moved R13 0.17 mm to (146.4, 138.8)
Connections:
- net A0_LF renamed LEFT_FRONT_ADC
- net A1_RD renamed RIGHT_DIAG_ADC
- net A2_LD renamed LEFT_DIAG_ADC
- net A3_RF renamed RIGHT_FRONT_ADC
- net GPIO_LED renamed SENSOR_LED
Routing:
- net GND: track 43.1 -> 45.2 mm
- net Net-(FLED2-A): track 19.2 -> 20.8 mm
- net LEFT_DIAG_ADC: track 28.5 -> 27.5 mm
- net RIGHT_FRONT_ADC: track 39.8 -> 40.7 mm
- net LEFT_FRONT_ADC: track 47.7 -> 46.8 mm
- net SENSOR_LED: track 3.97 -> 3.08 mm
Other:
- outline, holes or cut-outs redrawn
