File: MouseSMDUKMARSAdvancedBoard/MouseSMDUKMARSAdvancedBoard.kicad_sch (KiCad schematic)
At the start: 33 parts, among them J1 Conn_01x10

Commit message: Updates based on feedback
Parts:
- FET1, FET2: value BSH108,215 -> PMV45EN2; footprint Package_TO_SOT_SMD:SOT-23 -> Package_TO_SOT_SMD:SOT-23_Handsoldering; symbol Transistor_FET:BF545A -> PB_Library:PMV45EN2
- LDPD1, LFPD1, RDPD1, RFPD2: symbol Device:D_Photo -> Sensor_Optical:BPW40
- TR1, TR2: footprint Package_TO_SOT_SMD:SOT-23 -> Package_TO_SOT_SMD:SOT-23_Handsoldering
Connections:
- net at R2.2, R4.1, TR2.3 (C): now also FET2.1 (G); no longer FET2.3 (G)
- net at C2.1, FLED2.2 (A), R7.2: no longer FLED1.2 (A)
- net at R8.1, TR2.1 (B): now also FET2.2 (S); no longer FET2.1 (S)
- net at R6.1, TR1.1 (B): now also FET1.2 (S); no longer FET1.1 (S)
- net at R1.2, R3.1, TR1.3 (C): now also FET1.1 (G); no longer FET1.3 (G)
- net at C1.1, DLED2.2 (A), R5.2: no longer DLED1.2 (A)
- net +3.3V renamed Vcc
- net +9V renamed Vbatt
- new net: FLED1.2 (A), FLED2.1 (K)
- new net: DLED1.1 (K), FET1.3 (D)
- new net: DLED1.2 (A), DLED2.1 (K)
- new net: FET2.3 (D), FLED1.1 (K)
Other:
- moved on the sheet: DLED1, DLED2, FLED1, FLED2

Commit message: Sort of ready for JLCPCB
Parts:
- added H1, H2: 3.2mm, MountingHole:MountingHole_3.2mm_M3_Pad, symbol Mechanical:MountingHole_Pad
Connections:
- net GND: now also H1.1, H2.1
- net A0_LF renamed LEFT_FRONT_ADC
- net A1_RD renamed RIGHT_DIAG_ADC
- net A2_LD renamed LEFT_DIAG_ADC
- net A3_RF renamed RIGHT_FRONT_ADC
- net GPIO_LED renamed SENSOR_LED
Other:
- note added: "Mounting Holes"
