File: SSEverythingMainBoard/SSEverythingMainBoard.kicad_pcb (KiCad board)
At the start: 2 copper layers, 99.1 x 81.3 mm, 58 parts, among them J1 CONN_06SILK_FEMALE_PTH, J2 CONN_06SILK_FEMALE_PTH, J3 POWER, J4 Switch, J5 Conn_01x02, J6 Conn_01x05, M1 Left MOTOR, M2 Right MOTOR, SW1 TACT_SW, U1 DFRobot_DC_Controller

Commit message: Send boards to JLCPCB
Parts:
- added C10: 0.1uF, Capacitor_SMD:C_0805_2012Metric_Pad1.18x1.45mm_HandSolder, F.Cu at (133.0, 67.3)
- added C11: 10uF, Capacitor_SMD:C_0805_2012Metric_Pad1.18x1.45mm_HandSolder, F.Cu at (161.4, 95.7)
- added C12: 0.1uF, Capacitor_SMD:C_0805_2012Metric_Pad1.18x1.45mm_HandSolder, F.Cu at (161.4, 97.9)
- added C7: 0.1uF, Capacitor_SMD:C_0805_2012Metric_Pad1.18x1.45mm_HandSolder, F.Cu at (146.7, 134.3)
- added C8: 0.1uF, Capacitor_SMD:C_0805_2012Metric_Pad1.18x1.45mm_HandSolder, F.Cu at (161.6, 116.9)
- added C9: 10uF, Capacitor_SMD:C_0805_2012Metric_Pad1.18x1.45mm_HandSolder, F.Cu at (133.0, 69.4)
- added G***: LOGO, PBFootPrintLibrary:MicroPythonLogo, F.Cu at (151.2, 105.5)
- added G***: LOGO, PBFootPrintLibrary:MicroPythonLogo, B.Cu at (151.1, 105.6)
- moved SW1 94.2 mm to (78.8, 129.2), turned to 180 degrees
- moved GROUND2 86.4 mm to (124.7, 79.3)
- moved GROUND1 67.4 mm to (127.6, 133.3)
- moved J5 58.9 mm to (88.3, 118.3)
- moved R8 40.3 mm to (130.2, 78.4)
- moved R18 40.3 mm to (73.3, 135.5), turned to 90 degrees
- moved D3 39.9 mm to (71.0, 140.7), turned to -90 degrees
- moved J6 37.4 mm to (83.3, 118.7), turned to -90 degrees
- moved R17 35.5 mm to (73.7, 140.3), turned to -90 degrees
- moved R4 34.4 mm to (140.7, 79.7)
- moved R2 31.0 mm to (140.7, 82.3)
- moved D5 30.8 mm to (140.1, 92.6), turned to 0 degrees
- moved R9 30.4 mm to (130.7, 74.8), turned to -90 degrees
- moved TR2 30.2 mm to (135.1, 79.6)
- moved R3 30.1 mm to (147.6, 80.8), turned to -90 degrees
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- renumbered RFPD1 to LFPD1, LFPD1 to RFPD1
Connections:
- A1 pad 19: RIGHT_DIAG_ADC -> LEFT_FRONT_ADC
- A1 pad 20: RIGHT_FRONT_ADC -> LEFT_DIAG_ADC
- A1 pad 21: LEFT_FRONT_ADC -> RIGHT_DIAG_ADC
- A1 pad 22: LEFT_DIAG_ADC -> RIGHT_FRONT_ADC
- A1 pad 5: RIGHT_Motor_PWM -> LEFT_MOTOR_Dir
- A1 pad 6: LEFT_Motor_PWM -> LEFT_MOTOR_PWM
- A1 pad 7: LEFT_Motor_Dir -> RIGHT_MOTOR_PWM
- A1 pad 8: RIGHT_Motor_Dir -> RIGHT_MOTOR_Dir
- C1 pad 1: Net-(DLED1-A) -> Net-(DLED2-A)
- DLED2 pad 1: Net-(DLED2-K) -> Net-(DLED1-A)
- DLED2 pad 2: Net-(DLED1-K) -> Net-(DLED2-A)
- FET1 pad 3: Net-(DLED2-K) -> Net-(DLED1-K)
- J2 pad 2: LEFT_ENC_A -> LEFT_ENC_B
- J2 pad 3: LEFT_ENC_B -> LEFT_ENC_A
- LFPD1 pad 2: RIGHT_FRONT_ADC -> LEFT_FRONT_ADC
- R5 pad 2: Net-(DLED1-A) -> Net-(DLED2-A)
- RFPD1 pad 2: LEFT_FRONT_ADC -> RIGHT_FRONT_ADC
Routing:
- net Net-(LFPD1-C): track 0.00 -> 133.2 mm
- net Net-(FLED1-K): track 0.00 -> 116.9 mm
- net Vcc: track 91.5 -> 200.8 mm, vias 0 -> 3
- net Vbatt: track 60.8 -> 155.8 mm
- net RIGHT_FRONT_ADC: track 46.3 -> 128.0 mm
- net LEFT_DIAG_ADC: track 45.7 -> 123.7 mm
- net RIGHT_DIAG_ADC: track 45.9 -> 117.6 mm
- net Net-(A1-D13/SCK): track 0.00 -> 65.2 mm, vias 0 -> 1
- net GND: track 6.60 -> 64.1 mm, vias 0 -> 14
- net GPIO_DIAG: track 46.8 -> 103.5 mm
- net Net-(A1-D0/RX): track 0.00 -> 51.0 mm, vias 0 -> 3
- net SENSOR_LED: track 48.3 -> 98.9 mm
- net Net-(DLED1-A): track 0.00 -> 49.2 mm
- net Net-(LDPD1-C): track 0.00 -> 48.7 mm
- net LEFT_MOTOR_PWM: track 8.41 -> 57.0 mm
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Other:
- board text added: "A4"
- board text added: "A5"
